File: hardware/mao/power.kicad_sch (KiCad schematic)
At the start: 35 parts, among them J101 USB-C, J102 BAT, Q101 AO3401A, Q102 2N7002, U101 TPD2E2U06, U102 BQ25185DLHR, U103 MAX17048G+T10, U104 TPS62840DLCR, U105 TPS22916CYFPR

Commit message: A1: USB D+/D- as one pair on F over the L2 ground (design review 2026-10-06, finding 3)
The router had D+ on F but D- down B (x 0.2) across the L3 VBUS / +3V3 split under the receptacle. Both lines now run
on F as a designed edge-coupled pair, w 0.15 / gap 0.25 (~90 ohm differential on JLC04161H-1080; project.py), from
the receptacle's F join / one D- via, in line through the ESD array (its two identical channels swap: pin 3 D-,
pin 5 D+), round the face switch's east side and into the 22R R216/R215 (route_local.USB_PAIR). To make room the I2C
data line turns 0.35 mm earlier and the I2C clock's B->L3 via north of the 22R moves 0.9 mm (route_review.py 3).
Pair: D+ 34.4 mm F + 1.1 mm B (contact stubs), D- 31.7 mm F + 3.9 mm B. DRC 0 / 0 / 0, planes continuous.

Co-Authored-By: Claude Opus 5.5 <noreply@anthropic.com>
Connections:
- net USB_C_DN: now also U101.3; no longer U101.5
- net USB_C_DP: now also U101.5; no longer U101.3
Changed lines of the file:
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@@
 			)
 		)
-		(property "Description" "2-ch ESD, 1.5 pF, IEC 61000-4-2 level 4"
+		(property "Description" "2-ch ESD, 1.5 pF, IEC 61000-4-2 level 4; the two identical channels take D- (pin 3) and D+ (pin 5) so the pair passes through them in the order the module wants (design review 2026-10-06)"
 			(at 121.92 36.83 0)
 			(effects
@@
 		(at 129.54 39.37)
 	)
-	(global_label "USB_C_DP"
+	(global_label "USB_C_DN"
 		(shape bidirectional)
 		(at 114.3 34.29 180)
@@
 		)
 	)
-	(global_label "USB_C_DN"
+	(global_label "USB_C_DP"
 		(shape bidirectional)
 		(at 114.3 39.37 180)
